File: ISA68618.kicad_sch (KiCad schematic)
At the start: 4 parts

Commit message: ISA68030 - update
Parts:
- added U? (x2): 74ACT04, symbol 74xx:74LS04
- added U?: 74ACT08, symbol 74xx:74LS08
- added U?: 74LS161, symbol 74xx:74LS161
- U? (x2): value 74LS04 -> 74ACT04
Connections:
- net CA21: now also U?.5; no longer U?.3
- net at U?.13: now also U?.6; no longer U?.4
- net GND: now reaches U?.20 (GND)
- net GND: now also U?.3 (D0), U?.4 (D1), U?.6 (D3), U?.8 (GND)
- net IRQ4: now reaches U?.21 (IRQ)
- net at U?.32 (X1/CLK): now also U?.2, U?.9 (~{PE})
- net RESETN: now reaches U?.34 (RESET)
- net IACK4: now reaches U?.37 (IACK)
- net +5V: now reaches U?.40 (VCC)
- net +5V: now also U?.1 (~{MR}), U?.10 (CET), U?.16 (VCC), U?.5 (D2), U?.7 (CEP)
- net CA12: no longer names the net of U?.2
- net CA12: now also U?.4
- net CS681N: no longer names the net of U?.35 (CS), U?.9
- new net: U?.1, U?.3
- new net: U?.1, U?.12 (Q2)
- new net: U?.11 (Q3), U?.2
- new net BANK0: U?.3
- new net GCLK: U?.2 (CP)
Other:
- note added: "$00DFExxx"
- note added: "3.6409 MHz"
- moved on the sheet: U?, U?A, U?C
