File: CMod.kicad_sch (KiCad schematic)
At the start: 2 parts

Commit message: ISA68030 - update
Parts:
- added C? (x10): 0.1u, symbol Device:C
- added R?: 3k3, symbol Device:R
- added U18: 74ACT32, symbol 74xx:74LS32
- added U40: 74LVC04, symbol 74xx:74LS04
- added U41: 74F521, symbol MyLib:74F521
- gave numbers to parts that had none: 2
Connections:
- net +3.3V: now also R?.1, U40.14 (VCC)
- net CRW: now also U18.5
- net GND: now also C?.2, C?.2, C?.2, C?.2, C?.2, C?.2, C?.2, C?.2, C?.2, C?.2, U40.7 (GND), U41.1 (A=Bin), U41.10 (GND), U41.12 (B4), U41.14 (B5), U41.16 (B6), U41.17 (A7), U41.18 (B7), U41.3 (B0), U41.5 (B1), U41.7 (B2), U41.9 (B3)
- net CMDBEN: now reaches U42.19 (CE)
- net CMDBEN: now also U40.1, U41.19 (A=BOut)
- net at U43.22 (PIO22): now also U40.2
- net at U43.23 (PIO23): now also U40.4
- net BERRE: now reaches U43.33 (PIO33)
- net at U43.34 (PIO34): now also U40.8
- net at U43.35 (PIO35): now also U40.5
- net BANK0ACK: now reaches U43.36 (PIO36)
- net BANK0ACK: now also R?.2
- net RTS: now reaches U43.37 (PIO37)
- net CTS: now reaches U43.38 (PIO38)
- net RxD: now reaches U43.39 (PIO39)
- net TxD: now reaches U43.40 (PIO40)
- new net: U18.6, U40.3
- new net +5V: C?.1, C?.1, C?.1, C?.1, C?.1, C?.1, C?.1, C?.1, C?.1, C?.1, U41.20 (VCC)
- new net BANK0: U41.15 (A6)
- new net CA19: U41.2 (A0)
- new net CA20: U41.4 (A1)
- new net CA21: U41.6 (A2)
- new net CA22: U41.8 (A3)
- new net CA23: U41.11 (A4)
- new net CAS: U41.13 (A5)
- new net CDS: U18.4
- new net IACK4: U40.9
- new net IRQ4: U40.6
Other:
- company: (none) -> Finitron
- title: (none) -> ISA68030 Boot ROM, Keyboard, Mouse
- moved on the sheet: U42, U43

Commit message: ISA68030 - update
Parts:
- added C?: 0.047u, Capacitor_THT:C_Disc_D3.8mm_W2.6mm_P2.50mm, symbol ISA_FPGA_v2-rescue:CP1-Device
- added C?: 100u, Capacitor_THT:CP_Radial_D8.0mm_P3.80mm, symbol ISA_FPGA_v2-rescue:CP1-Device
- added C?: 10u, symbol Device:C
- added C?: 10u, Capacitor_THT:CP_Radial_D5.0mm_P2.50mm, symbol ISA_FPGA_v2-rescue:CP1-Device
- added C?: 220u, Capacitor_THT:CP_Radial_D8.0mm_P3.80mm, symbol ISA_FPGA_v2-rescue:CP1-Device
- added C?: 0.047u, Capacitor_THT:C_Disc_D5.0mm_W2.5mm_P5.00mm, symbol ISA_FPGA_v2-rescue:CP1-Device
- added D?: DIODE, symbol pspice:DIODE
- added J?: AudioJack2, Connector_Audio:Jack_3.5mm_CUI_SJ1-3533NG_Horizontal, symbol Connector:AudioJack2
- added R? (x2): 5k1, Resistor_THT:R_Axial_DIN0207_L6.3mm_D2.5mm_P7.62mm_Horizontal, symbol VGA_V11-cache:R
- added R? (x2): 3k3, symbol Device:R
- added R?: 10, Resistor_THT:R_Axial_DIN0207_L6.3mm_D2.5mm_P7.62mm_Horizontal, symbol VGA_V11-cache:R
- added U44: VDIP2-32, Package_DIP:DIP-32_W15.24mm_Socket, symbol MyLib:VDIP2-32
- added U45: LM386, Package_DIP:DIP-8_W7.62mm_Socket, symbol Amplifier_Audio:LM386
- U40: footprint (none) -> Package_DIP:DIP-14_W7.62mm_Socket
- U41: footprint (none) -> Package_DIP:DIP-20_W7.62mm_Socket
- U43: footprint (none) -> Package_DIP:DIP-48_W15.24mm_Socket
Connections:
- net +3.3V: now also R?.1, R?.1
- net +5V: now also C?.1, D?.1 (K), U44.1 (+5V)
- net CTS: now also U44.9 (RTS)
- net GND: now also U43.25 (GND), C?.2, C?.2, C?.2, C?.2, J?.S, R?.1, U44.18 (GND), U44.4 (GND), U44.5 (GND), U44.7 (GND), U45.2 (-), U45.4 (GND)
- net RTS: now also U44.10 (CTS)
- net RxD: now also U44.6 (TxD)
- net TxD: now also U44.8 (RxD)
- net at U43.24 (VU): now also D?.2 (A)
- net AUD: now reaches U43.30 (PIO30)
- net AUD: now also C?.1, R?.2
- net VPROG: now reaches U43.31 (PIO31)
- net VPROG: now also R?.2, U44.23 (PROG)
- net VRESET: now reaches U43.32 (PIO32)
- net VRESET: now also R?.2, U44.22 (RESET)
- new net: R?.1, R?.2, U45.3 (+)
- new net: C?.1, U45.1 (GAIN)
- new net: C?.2, U45.8 (GAIN)
- new net: C?.2, J?.T
- new net: C?.1, R?.2, U45.5
- new net: C?.1, R?.1
- new net +12V: C?.1, U45.6 (V+)
- no-connect marks 0 -> 10
Other:
- note added: "USB Host for keyboard / mouse"
- title: ISA68030 Boot ROM, Keyboard, Mouse -> ISA68030 Boot ROM, Keyboard, Mouse, Audio

Commit message: ISA68030 - update
Parts:
- removed U18: 74ACT32, symbol 74xx:74LS32
- added unit 5 of U40
- added unit 6 of U40
Connections:
- net GND: now also U40.11, U40.13
- net CXRW: now reaches U40.3
- no-connect marks 10 -> 12

Commit message: ISA68030 - update
Connections:
- net CLK525: now reaches U43.29 (PIO29)
Changed lines of the file:
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@@
+    (stroke (width 0) (type default) (color 0 0 0 0))
+  )
+  (wire (pts (xy 144.78 100.33) (xy 138.43 100.33))
     (stroke (width 0) (type default) (color 0 0 0 0))
   )
@@
     (stroke (width 0) (type default) (color 0 0 0 0))
   )
+  (wire (pts (xy 138.43 100.33) (xy 138.43 91.44))
+    (stroke (width 0) (type default) (color 0 0 0 0))
+  )
   (wire (pts (xy 110.49 68.58) (xy 104.14 68.58))
     (stroke (width 0) (type default) (color 0 0 0 0))
@@
   )
   (bus (pts (xy 101.6 55.88) (xy 101.6 53.34))
+    (stroke (width 0) (type default) (color 0 0 0 0))
+  )
+  (wire (pts (xy 138.43 91.44) (xy 132.08 91.44))
     (stroke (width 0) (type default) (color 0 0 0 0))
   )
@@
       (effects (font (size 1.27 1.27)) (justify left) hide)
     )
+  )
+  (global_label "CLK525" (shape output) (at 144.78 100.33 0) (fields_autoplaced)
+    (effects (font (size 1.27 1.27)) (justify left))
+    (property "Intersheet References" "${INTERSHEET_REFS}" (id 0) (at 154.3898 100.2506 0)
+      (effects (font (size 1.27 1.27)) (justify left) hide)
+    )
