File: ClockGen.kicad_sch (KiCad schematic)
At the start: 5 parts, among them U1 74ACT04, U18 74ACT32, U50 ICS525R-02, U51 74LS273, X1 32.768MHz

Commit message: ISA68030 - update
Parts:
- added C? (x2): 0.01u, symbol Device:C
- U51: value 74LS273 -> 74ACT273
- X1: value 32.768MHz -> 19.608 MHz
Connections:
- net +5V: now also C?.1, C?.2
- net GND: now also C?.1, C?.2
- net at U1.3: now also U51.16 (Q6); no longer U51.15 (Q5)
- net at U1.4: now also U50.16 (V6); no longer U50.15 (V5)
- net at U1.1, U50.21 (CLK): no longer U18.4, U18.5
- net at U50.22 (REF): now also U18.4, U18.5
- new net: U50.15 (V5), U51.15 (Q5)
- no-connect marks 2 -> 1
Other:
- note added: "Caps, one on each side as close to power as possible"
- note added: "Default clock is 9.804 MHz"
- note removed: "Default clock is 8.192 MHz"
- moved on the sheet: U18B, U1A, U1B, U50, U51, X1
