File: ISA68010.kicad_sch (KiCad schematic)
At the start: 56 parts, among them J1 Bus_ISA_16bit, U1 74ACT04, U10 DS1813, U11 68030, U12 74ACT245, U13 74ACT245, U14 74ACT245, U15 74ACT245, U16 74ACT245, U17 74ACT245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

Commit message: ISA68030 - update
Parts:
- added R? (x2): 3k3, symbol Device:R
Connections:
- net AS is gone; now on net XAS: U17.14 (B4)
- net +5V: now also R?.1, R?.1
- net XAS: now also R?.2
- net XBERR: now also R?.2
- net +12V: now reaches J1.9 (+12V)
- no-connect marks 17 -> 35
Other:
- removed sheet 68681

Commit message: ISA68030 - update
Parts:
- removed U3: 74ACT08, symbol 74xx:74LS08
- added unit 4 of U18
- added unit 3 of U18
- added unit 3 of U4
- U18: footprint (none) -> Package_DIP:DIP-14_W7.62mm_Socket
Connections:
- net BERR: now also U4.8
- net CACHE: now also U11.L1 (CIIN*)
- net GND: now also U18.10, U18.12, U18.13, U18.4, U18.5, U18.9
- net XBERR: now also U4.11
- net at U1.6, U2.10 (CET), U2.7 (CEP): now also U4.10, U4.9
- no-connect marks 35 -> 38
Other:
- moved on the sheet: C?, R?, U18B, U18E, U1E, U4D, U9, U?C

Commit message: ISA68030 - update
Connections:
- no-connect marks 38 -> 39
Changed lines of the file:
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@@
   (no_connect (at 134.62 152.4))
   (no_connect (at 134.62 149.86))
+  (no_connect (at 134.62 312.42))
   (no_connect (at 101.6 181.61))
   (no_connect (at 101.6 194.31))
@@
       (reference "#PWR?") (unit 1) (value "+3.3V") (footprint "")
     )
+    (path "/9957abb0-b5bf-42c3-97c1-5fe27718e073/08c5fb25-223a-496d-8f1c-63d5b8bf9b68"
+      (reference "#PWR?") (unit 1) (value "GND") (footprint "")
+    )
     (path "/0b2bdb57-5ea8-4afa-a121-2df9c8d45827"
       (reference "#PWR?") (unit 1) (value "+5V") (footprint "")
@@
       (reference "#PWR?") (unit 1) (value "GND") (footprint "")
     )
+    (path "/d75377c2-8e80-44be-a5c5-a22e3859d2fe/b86c57f1-494b-4f41-9f03-740ea0ed95dc"
+      (reference "#PWR?") (unit 1) (value "GND") (footprint "")
+    )
     (path "/9957abb0-b5bf-42c3-97c1-5fe27718e073/b9188883-2ada-4b80-85fa-606412e00e0d"
       (reference "#PWR?") (unit 1) (value "GND") (footprint "")
@@
       (reference "U23") (unit 4) (value "74ACT04") (footprint "")
     )
+    (path "/9957abb0-b5bf-42c3-97c1-5fe27718e073/ed1406d1-2ecb-4ae5-a8b1-17c93b8a581c"
+      (reference "U23") (unit 5) (value "74ACT04") (footprint "")
+    )
+    (path "/9957abb0-b5bf-42c3-97c1-5fe27718e073/7ded3bd6-e352-433f-9e56-a4f3d1923642"
+      (reference "U23") (unit 6) (value "74ACT04") (footprint "")
+    )
     (path "/9957abb0-b5bf-42c3-97c1-5fe27718e073/0a9a0874-7a46-4bfe-a3bd-f2f07252563f"
       (reference "U23") (unit 7) (value "74ACT04") (footprint "")
@@
       (reference "U40") (unit 4) (value "74LVC04") (footprint "Package_DIP:DIP-14_W7.62mm_Socket")
     )
+    (path "/d75377c2-8e80-44be-a5c5-a22e3859d2fe/28c1f339-fa49-4bfa-8cc0-e3b83fc0a3dc"
+      (reference "U40") (unit 5) (value "74LVC04") (footprint "Package_DIP:DIP-14_W7.62mm_Socket")
+    )
+    (path "/d75377c2-8e80-44be-a5c5-a22e3859d2fe/7522616f-a6f9-467d-861a-e19a6414a9dd"
+      (reference "U40") (unit 6) (value "74LVC04") (footprint "Package_DIP:DIP-14_W7.62mm_Socket")
+    )
     (path "/d75377c2-8e80-44be-a5c5-a22e3859d2fe/7c708fbe-1747-4d48-81dd-5a02fbb56120"

Commit message: ISA68030 - update
Parts:
- removed unit 1 of U1
- removed unit 2 of U1
- removed U18: 74ACT32, Package_DIP:DIP-14_W7.62mm_Socket, symbol 74xx:74LS32
- removed X?: 32.768MHz, Oscillator:Oscillator_DIP-8, symbol Oscillator:CXO_DIP8
- U1: footprint (none) -> Package_DIP:DIP-14_W7.62mm_Socket
Connections:
- net CA24: now also U17.2 (A0)
- net CA25: now also U17.3 (A1)
- net CA26: now also U17.4 (A2)
- net CA27: now also U17.5 (A3)
- net CAS: now also U17.7 (A5); no longer U17.6 (A4)
- net CFC0: no longer U17.2 (A0)
- net CFC1: no longer U17.3 (A1)
- net CFC2: no longer U17.4 (A2)
- net CSIZ0: now also U17.8 (A6); no longer U17.7 (A5)
- net CSIZ1: now also U17.9 (A7); no longer U17.8 (A6)
- net CXRW: now also U17.6 (A4); no longer U17.5 (A3)
- net RW: now also U17.14 (B4); no longer U17.15 (B3)
- net SIZ0: now also U17.12 (B6); no longer U17.13 (B5)
- net SIZ1: now also U17.11 (B7); no longer U17.12 (B6)
- net XAS: now also U17.13 (B5); no longer U17.14 (B4)
- net LA24: now reaches J1.81 (SBHE)
- net LA24: now also U17.18 (B0)
- net FC0 renamed LA25
- net LA25: now also U17.17 (B1); no longer U17.18 (B0)
- net FC1 renamed LA26
- net LA26: now also U17.16 (B2); no longer U17.17 (B1)
- net FC2 renamed LA27
- net LA27: now also U17.15 (B3); no longer U17.16 (B2)
- no-connect marks 39 -> 35
Other:
- added sheet ClockGen (ClockGen.kicad_sch)
- moved on the sheet: D?, R?, RN?, U1F

Commit message: ISA68030 - update
Connections:
- net +5V: no longer U8.12 (B4), U8.14 (B5), U8.16 (B6), U8.18 (B7), U8.5 (B1), U8.7 (B2), U8.9 (B3)
- net CA24: no longer R?.2, U8.2 (A0)
- net CA25: no longer U8.4 (A1)
- net CA26: no longer U8.6 (A2)
- net CA27: no longer U8.8 (A3)
- net GND: now also U8.12 (B4), U8.2 (A0), U8.4 (A1), U8.5 (B1), U8.6 (A2), U8.7 (B2), U8.8 (A3), U8.9 (B3)
- new net: R?.2, U8.14 (B5), U8.16 (B6), U8.18 (B7)
Other:
- note added: "ISA BUS @$Exxxxxxx"
- note removed: "ISA BUS @$FExxxxxx"
- moved on the sheet: R?

Commit message: ISA68030 - update
Parts:
- removed R?: 3k3, symbol Device:R
- removed RN?: 3k3, Resistor_THT:R_Array_SIP5, symbol Device:R_Network04
- added R?: 3k3, symbol Device:R
- added RN?: 3k3, Resistor_THT:R_Array_SIP9, symbol Device:R_Network08
Connections:
- net +5V: now also R?.1, RN?.1 (common)
- net CA27: no longer U17.5 (A3)
- net CA28: now also R?.2
- net CAS: now also RN?.2 (R1)
- net CDIS: now also RN?.5 (R4)
- net CDS: now also U17.5 (A3), RN?.3 (R2)
- net CRW: now also U17.6 (A4), RN?.4 (R3)
- net CXRW: no longer U17.6 (A4)
- net DONE: now also RN?.7 (R6)
- net HALT: now also RN?.8 (R7)
- net MMUDIS: now also RN?.6 (R5)
- net RESETN: now also RN?.9 (R8)
- net XAVEC: now also J1.19 (~{REFRESH}); no longer J1.89 (~{MEMR})
- net at U8.14 (B5), U8.16 (B6), U8.18 (B7): now also R?.2; no longer R?.2
- net LA27: no longer names the net of J1.88 (LA17)
- net LA27: no longer U17.15 (B3)
- new net XDS: J1.89 (~{MEMR}), U17.15 (B3)
Other:
- moved on the sheet: R?
