File: ISA68030_SRAM.kicad_sch (KiCad schematic)
At the start: 16 parts

Commit message: ISA68030 - update
Parts:
- added C? (x10): 0.1u, symbol Device:C
- added unit 7 of U23
- added unit 4 of U23
- U23: renamed from U?; value 74LS04 -> 74ACT04
- U23: renamed from U?; value 74F04 -> 74ACT04
- U24: renamed from U?; value 74F175 -> 74ACT175
- gave numbers to parts that had none: 11
Connections:
- net +5V: now also U28.1 (I1/CLK), C?.1, C?.1, C?.1, C?.1, C?.1, C?.1, C?.1, C?.1, C?.1, C?.1, U23.14 (VCC)
- net BANK1: now also U23.3, U23.9; no longer U23.1
- net CAS: now also U23.5; no longer U23.1
- net GND: now also U28.8 (I8), U28.9 (I9), C?.2, C?.2, C?.2, C?.2, C?.2, C?.2, C?.2, C?.2, C?.2, C?.2, U23.7 (GND)
- net at U24.1 (~{Mr}): now also U23.6; no longer U23.2
- net at U24.13 (D3): now also U23.4; no longer U23.2
- new net CACHE: U23.8
- no-connect marks 0 -> 4

Commit message: ISA68030 - update
Parts:
- added unit 6 of U23
- added unit 5 of U23
Connections:
- net GND: now also U23.11, U23.13
- no-connect marks 4 -> 6
Other:
- moved on the sheet: U23B, U23C, U24

Commit message: ISA68030 - update
Parts:
- added R?: 3k3, symbol Device:R
Connections:
- net +3.3V: now also R?.1
- net WE0: now also U33.20 (WE0), U33.27 (WE1); no longer U30.20 (WE0), U30.27 (WE1)
- net WE1: now also U32.20 (WE0), U32.27 (WE1); no longer U31.20 (WE0), U31.27 (WE1)
- net WE2: now also U31.20 (WE0), U31.27 (WE1); no longer U32.20 (WE0), U32.27 (WE1)
- net WE3: now also U30.20 (WE0), U30.27 (WE1); no longer U33.20 (WE0), U33.27 (WE1)
- net PU2: now reaches U22.1 (A->B)
- net PU2: now also U20.1 (A->B), U21.1 (A->B), R?.2
- no-connect marks 6 -> 10
Changed lines of the file:
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@@
   (junction (at 157.48 160.02) (diameter 0) (color 0 0 0 0)
   )
+  (junction (at 46.99 68.58) (diameter 0) (color 0 0 0 0)
+  )
   (junction (at 237.49 100.33) (diameter 0) (color 0 0 0 0)
   )
@@
   (no_connect (at 309.88 153.67))
   (no_connect (at 309.88 156.21))
+  (no_connect (at 91.44 162.56))
+  (no_connect (at 91.44 165.1))
+  (no_connect (at 66.04 165.1))
+  (no_connect (at 66.04 162.56))
   (no_connect (at 316.23 151.13))
   (no_connect (at 73.66 248.92))
@@
     (stroke (width 0) (type default) (color 0 0 0 0))
   )
+  (wire (pts (xy 46.99 68.58) (xy 66.04 68.58))
+    (stroke (width 0) (type default) (color 0 0 0 0))
+  )
   (bus (pts (xy 156.21 35.56) (xy 156.21 53.34))
     (stroke (width 0) (type default) (color 0 0 0 0))
@@
     (stroke (width 0) (type default) (color 0 0 0 0))
   )
+  (wire (pts (xy 66.04 170.18) (xy 57.15 170.18))
+    (stroke (width 0) (type default) (color 0 0 0 0))
+  )
   (wire (pts (xy 163.83 55.88) (xy 158.75 55.88))
     (stroke (width 0) (type default) (color 0 0 0 0))
@@
     (stroke (width 0) (type default) (color 0 0 0 0))
   )
+  (wire (pts (xy 46.99 62.23) (xy 46.99 68.58))
+    (stroke (width 0) (type default) (color 0 0 0 0))
+  )
   (wire (pts (xy 284.48 99.06) (xy 281.94 99.06))
     (stroke (width 0) (type default) (color 0 0 0 0))
@@
     (stroke (width 0) (type default) (color 0 0 0 0))
   )
+  (wire (pts (xy 46.99 119.38) (xy 46.99 68.58))
+    (stroke (width 0) (type default) (color 0 0 0 0))
+  )
   (wire (pts (xy 173.99 52.07) (xy 173.99 50.8))
     (stroke (width 0) (type default) (color 0 0 0 0))
@@
     (stroke (width 0) (type default) (color 0 0 0 0))
   )
+  (wire (pts (xy 46.99 119.38) (xy 66.04 119.38))
+    (stroke (width 0) (type default) (color 0 0 0 0))
+  )
   (bus (pts (xy 99.06 114.3) (xy 99.06 111.76))
     (stroke (width 0) (type default) (color 0 0 0 0))
@@
     (effects (font (size 1.27 1.27)) (justify left bottom))
   )
-  (label "WE0" (at 143.51 101.6 180)
+  (label "WE3" (at 143.51 101.6 180)
     (effects (font (size 1.27 1.27)) (justify right bottom))
   )
@@
     (effects (font (size 1.27 1.27)) (justify left bottom))
   )
-  (label "WE2" (at 237.49 100.33 0)
+  (label "WE1" (at 237.49 100.33 0)
     (effects (font (size 1.27 1.27)) (justify left bottom))
   )
@@
     (effects (font (size 1.27 1.27)) (justify right bottom))
   )
+  (label "PU2" (at 49.53 119.38 0)
+    (effects (font (size 1.27 1.27)) (justify left bottom))
+  )
   (label "RA18" (at 207.01 96.52 0)
     (effects (font (size 1.27 1.27)) (justify left bottom))
@@
     (effects (font (size 1.27 1.27)) (justify left bottom))
   )
-  (label "WE3" (at 284.48 100.33 0)
+  (label "WE0" (at 284.48 100.33 0)
     (effects (font (size 1.27 1.27)) (justify left bottom))
   )
@@
     (effects (font (size 1.27 1.27)) (justify left bottom))
   )
+  (label "PU2" (at 59.69 170.18 0)
+    (effects (font (size 1.27 1.27)) (justify left bottom))
+  )
   (label "CD10" (at 186.69 60.96 0)
     (effects (font (size 1.27 1.27)) (justify left bottom))
@@
     (effects (font (size 1.27 1.27)) (justify left bottom))
   )
-  (label "WE1" (at 193.04 101.6 180)
+  (label "WE2" (at 193.04 101.6 180)
     (effects (font (size 1.27 1.27)) (justify right bottom))
   )
@@
     (pin "1")
   )
+  (symbol (lib_id "Device:R") (at 46.99 58.42 0) (unit 1)
+    (in_bom yes) (on_board yes) (fields_autoplaced)
+    (property "Reference" "R?" (id 0) (at 48.768 57.5853 0)
+      (effects (font (size 1.27 1.27)) (justify left))
+    )
+    (property "Value" "3k3" (id 1) (at 48.768 60.1222 0)
+      (effects (font (size 1.27 1.27)) (justify left))
+    )
+    (property "Footprint" "" (id 2) (at 45.212 58.42 90)
+      (effects (font (size 1.27 1.27)) hide)
+    )
+    (property "Datasheet" "~" (id 3) (at 46.99 58.42 0)
+      (effects (font (size 1.27 1.27)) hide)
+    )
+    (pin "1")
+    (pin "2")
+  )
   (symbol (lib_id "power:GND") (at 66.04 124.46 0) (unit 1)
     (in_bom yes) (on_board yes) (fields_autoplaced)
@@
       (effects (font (size 1.27 1.27)) hide)
     )
+    (pin "1")
+  )
+  (symbol (lib_id "power:+3.3V") (at 46.99 54.61 0) (unit 1)
+    (in_bom yes) (on_board yes) (fields_autoplaced)
+    (property "Reference" "#PWR?" (id 0) (at 46.99 58.42 0)
+      (effects (font (size 1.27 1.27)) hide)
+    )
+    (property "Value" "+3.3V" (id 1) (at 46.99 51.0342 0))
+    (property "Footprint" "" (id 2) (at 46.99 54.61 0)
+      (effects (font (size 1.27 1.27)) hide)
+    )
+    (property "Datasheet" "" (id 3) (at 46.99 54.61 0)
+      (effects (font (size 1.27 1.27)) hide)
+    )
